File: atmega328p.sch (KiCad schematic (older format))
At the start: 6 parts, among them J6 ICSP, U6 ATMEGA328PB-AU, Y1 CSTNE16M0VH3L000R0

Commit message: Update to rev. F
Parts:
- C15, C16, C17: footprint Capacitors_SMD:C_0805_HandSoldering -> Capacitor_SMD:C_0805_2012Metric_Pad1.18x1.45mm_HandSolder
- U6: footprint Housings_QFP:TQFP-32_7x7mm_Pitch0.8mm -> Package_QFP:TQFP-32_7x7mm_P0.8mm
- Y1: footprint muRata-CSTNEx:CSTNEx -> Crystal:Resonator_SMD_muRata_CSTxExxV-3Pin_3.0x1.1mm
Changed lines of the file:
@@
 $Descr A4 11693 8268
 encoding utf-8
-Sheet 2 2
+Sheet 2 3
 Title "BKM-129X Compatible full, onboard MCU"
 Date ""
@@
 F 0 "U6" H 4750 4975 50  0000 R BNN
 F 1 "ATMEGA328PB-AU" H 4750 4900 50  0000 R BNN
-F 2 "Housings_QFP:TQFP-32_7x7mm_Pitch0.8mm" H 5100 2100 50  0001 L CIN
+F 2 "Package_QFP:TQFP-32_7x7mm_P0.8mm" H 5100 2100 50  0001 L CIN
 F 3 "" H 4850 3550 50  0001 C CNN
 	1    5150 3500
@@
 F 0 "Y1" H 7300 3175 50  0000 C CNN
 F 1 "CSTNE16M0VH3L000R0" H 7300 3100 50  0000 C CNN
-F 2 "muRata-CSTNEx:CSTNEx" H 7300 2950 50  0001 C CNN
+F 2 "Crystal:Resonator_SMD_muRata_CSTxExxV-3Pin_3.0x1.1mm" H 7300 2950 50  0001 C CNN
 F 3 "" H 7300 2950 50  0001 C CNN
 	1    7300 2950
@@
 	4950 5000 4950 5050
 Wire Wire Line
-	4950 5050 5050 5050
+	4950 5050 5000 5050
 Wire Wire Line
 	5000 5050 5000 5100
@@
 F 0 "C16" H 4675 1750 50  0000 L CNN
 F 1 "4.7uF" H 4675 1550 50  0000 L CNN
-F 2 "Capacitors_SMD:C_0805_HandSoldering" H 4688 1500 50  0001 C CNN
+F 2 "Capacitor_SMD:C_0805_2012Metric_Pad1.18x1.45mm_HandSolder" H 4688 1500 50  0001 C CNN
 F 3 "" H 4650 1650 50  0001 C CNN
 	1    4650 1650
@@
 F 0 "C15" H 4425 1750 50  0000 L CNN
 F 1 "1uF" H 4425 1550 50  0000 L CNN
-F 2 "Capacitors_SMD:C_0805_HandSoldering" H 4438 1500 50  0001 C CNN
+F 2 "Capacitor_SMD:C_0805_2012Metric_Pad1.18x1.45mm_HandSolder" H 4438 1500 50  0001 C CNN
 F 3 "" H 4400 1650 50  0001 C CNN
 	1    4400 1650
@@
 $EndComp
 Wire Wire Line
-	4400 1400 4400 1500
+	4400 1400 4400 1450
 Wire Wire Line
 	4650 1450 4650 1500
@@
 	4850 1900 5050 1900
 Wire Wire Line
-	5050 1450 5050 2000
+	5050 1450 5050 1900
 $Comp
 L bkm-129x-scart-vga-rescue:C C17
@@
 F 0 "C17" H 3625 2700 50  0000 L CNN
 F 1 "100nF" H 3625 2500 50  0000 L CNN
-F 2 "Capacitors_SMD:C_0805_HandSoldering" H 3638 2450 50  0001 C CNN
+F 2 "Capacitor_SMD:C_0805_2012Metric_Pad1.18x1.45mm_HandSolder" H 3638 2450 50  0001 C CNN
 F 3 "" H 3600 2600 50  0001 C CNN
 	1    3600 2600
@@
 	4400 1850 4650 1850
 Wire Wire Line
-	4400 1450 5050 1450
+	4400 1450 4650 1450
+Wire Wire Line
+	5000 5050 5050 5050
+Wire Wire Line
+	4400 1450 4400 1500
+Wire Wire Line
+	5050 1900 5050 2000
+Wire Wire Line
+	4650 1450 5050 1450
 $EndSCHEMATC
