File: bkm-129x-scart-vga.sch (KiCad schematic (older format))
At the start: 58 parts, among them J1 DB15_Female_HighDensity_Mount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, J2 SCART-F, J3 SJ1-353XNG, J5 Conn_02x32_Row_Letter_Last, Q1 DTC144EKA, Q2 MMBT3904, SW1 PBH4UEENAGX, SW2 PBH4UEENAGX, U1 ADG1611, U2 THS7374, U3 arduino-nano-v3, U4 74LVC125, U5 MIC3490-3.3

Commit message: Rev. C. Move to Kicad 5
Connections:
- net +3V3: now also U2.9 (BYPASS)
- net GND: no longer U2.9 (BYPASS)
Changed lines of the file:
@@
-$EndComp
-$Comp
-L power:GNDA #PWR06
-U 1 1 5E34BA4B
-P 6200 3000
-F 0 "#PWR06" H 6200 2750 50  0001 C CNN
-F 1 "GNDA" V 6200 2800 50  0000 C CNN
-F 2 "" H 6200 3000 50  0001 C CNN
-F 3 "" H 6200 3000 50  0001 C CNN
-	1    6200 3000
-	0    -1   -1   0
 $EndComp
 $Comp
@@
 Wire Wire Line
 	3500 6550 3700 6550
+$Comp
+L power:+3.3V #PWR?
+U 1 1 606A68E1
+P 6200 3000
+F 0 "#PWR?" H 6200 2850 50  0001 C CNN
+F 1 "+3.3V" V 6200 3250 50  0000 C CNN
+F 2 "" H 6200 3000 50  0001 C CNN
+F 3 "" H 6200 3000 50  0001 C CNN
+	1    6200 3000
+	0    1    1    0
+$EndComp
 $EndSCHEMATC

Commit message: Rev. D
Connections:
- net GND: no longer J1.9
- no-connect marks 52 -> 53
Changed lines of the file:
@@
-$EndComp
-$Comp
-L power:GNDA #PWR062
-U 1 1 5EECE0B0
-P 5900 1550
-F 0 "#PWR062" H 5900 1300 50  0001 C CNN
-F 1 "GNDA" V 5900 1350 50  0000 C CNN
-F 2 "" H 5900 1550 50  0001 C CNN
-F 3 "" H 5900 1550 50  0001 C CNN
-	1    5900 1550
-	1    0    0    -1
 $EndComp
 $Comp
@@
 	0    1    1    0
 $EndComp
+NoConn ~ 5900 1550
 $EndSCHEMATC

Commit message: Rev. D1
Parts:
- U5: value MIC3490-3.3 -> MIC3490-5.0
Connections:
- net GND: now also J1.5
Changed lines of the file:
@@
 P 4350 4100
 F 0 "U5" H 4350 4350 60  0000 C CNN
-F 1 "MIC3490-3.3" H 4350 3850 60  0000 C CNN
+F 1 "MIC3490-5.0" H 4350 3850 60  0000 C CNN
 F 2 "TO_SOT_Packages_SMD:SOT-23-5_HandSoldering" H 4150 4100 60  0001 C CNN
 F 3 "" H 4150 4100 60  0001 C CNN
@@
 	3500 6550 3700 6550
 $Comp
-L power:+3.3V #PWR?
+L power:+3.3V #PWR0101
 U 1 1 606A68E1
 P 6200 3000
-F 0 "#PWR?" H 6200 2850 50  0001 C CNN
+F 0 "#PWR0101" H 6200 2850 50  0001 C CNN
 F 1 "+3.3V" V 6200 3250 50  0000 C CNN
 F 2 "" H 6200 3000 50  0001 C CNN
@@
 $EndComp
 NoConn ~ 5900 1550
+$Comp
+L power:GNDA #PWR0102
+U 1 1 60F3D899
+P 6200 1550
+F 0 "#PWR0102" H 6200 1300 50  0001 C CNN
+F 1 "GNDA" V 6200 1350 50  0000 C CNN
+F 2 "" H 6200 1550 50  0001 C CNN
+F 3 "" H 6200 1550 50  0001 C CNN
+	1    6200 1550
+	1    0    0    -1
+$EndComp
 $EndSCHEMATC

Commit message: Rev. E
Parts:
- J5: footprint din-41612-64p-ra:DIN-41612-64P -> standard-pin-64p-ra:STANDARD-PIN-64P-RA
Changed lines of the file:
@@
 F 0 "J5" H 10300 4500 50  0000 C CNN
 F 1 "Conn_02x32_Row_Letter_Last" H 10300 1200 50  0000 C CNN
-F 2 "din-41612-64p-ra:DIN-41612-64P" H 10250 2900 50  0001 C CNN
+F 2 "standard-pin-64p-ra:STANDARD-PIN-64P-RA" H 10250 2900 50  0001 C CNN
 F 3 "" H 10250 2900 50  0001 C CNN
 	1    10250 2900

Commit message: Update to rev. F
Parts:
- C1, C10, C11, C12, C2, C3, C4, C5, C6, C9: footprint Capacitors_SMD:C_0805_HandSoldering -> Capacitor_SMD:C_0805_2012Metric_Pad1.18x1.45mm_HandSolder
- C13, C7, C8: footprint Capacitors_SMD:CP_Elec_6.3x5.3 -> Capacitor_SMD:CP_Elec_6.3x5.3
- D1, D2: footprint Diodes_SMD:D_0805 -> Diode_SMD:D_0805_2012Metric_Pad1.15x1.40mm_HandSolder
- Q1: footprint TO_SOT_Packages_SMD:SC-59_Handsoldering -> Package_TO_SOT_SMD:SC-59_Handsoldering
- Q2: footprint TO_SOT_Packages_SMD:SOT-23_Handsoldering -> Package_TO_SOT_SMD:SOT-23_Handsoldering
- R1, R10, R11, R12, R13, R14, R15, R16, R18, R19, R2, R20, R21, R22, R23, R24, R25, R26, R27, R28, R3, R32, R33, R34, R4, R5, R6, R7, R8, R9: footprint Resistors_SMD:R_0805_HandSoldering -> Resistor_SMD:R_0805_2012Metric_Pad1.20x1.40mm_HandSolder
- U1: footprint Housings_SSOP:TSSOP-16_4.4x5mm_Pitch0.65mm -> Package_SO:TSSOP-16_4.4x5mm_P0.65mm
- U2, U4: footprint Housings_SSOP:TSSOP-14_4.4x5mm_Pitch0.65mm -> Package_SO:TSSOP-14_4.4x5mm_P0.65mm
- U5: footprint TO_SOT_Packages_SMD:SOT-23-5_HandSoldering -> Package_TO_SOT_SMD:SOT-23-5_HandSoldering
